Commit message: Update path to be compliant with Baxter_isaac

File: ur_isaac/urdfs/ur_t42.urdf (robot description, URDF)
Before this commit: robot ur3, 20 links, 19 joints
Links:
- link finger_1_1: geometry collision mesh filename=/home/ubb/Documents/Baxter_isaac/ROS2/src/t42_gripper/t42_g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 scale=0.025400 0.025400 0.025400; visual mesh filename=/home/ubb/Documents/Baxter_isaac/ROS2/src/t42_gripper/t42_g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 scale=0.025400 0.025400 0.025400
- link finger_1_2: geometry collision mesh filename=/home/ubb/Documents/Baxter_isaac/ROS2/src/t42_gripper/t42_g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 scale=0.001 0.001 0.001; visual mesh filename=/home/ubb/Documents/Baxter_isaac/ROS2/src/t42_gripper/t42_g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 scale=0.001 0.001 0.001
- link finger_2_1: geometry collision mesh filename=/home/ubb/Documents/Baxter_isaac/ROS2/src/t42_gripper/t42_g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 scale=0.025400 0.025400 0.025400; visual mesh filename=/home/ubb/Documents/Baxter_isaac/ROS2/src/t42_gripper/t42_g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 scale=0.025400 0.025400 0.025400
- link finger_2_2: geometry collision mesh filename=/home/ubb/Documents/Baxter_isaac/ROS2/src/t42_gripper/t42_g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 scale=0.001 0.001 0.001; visual mesh filename=/home/ubb/Documents/Baxter_isaac/ROS2/src/t42_gripper/t42_g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 scale=0.001 0.001 0.001
- link swivel_1: geometry collision mesh filename=/home/ubb/Documents/Baxter_isaac/ROS2/src/t42_gripper/t42_g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 scale=0.001 0.001 0.001; visual mesh filename=/home/ubb/Documents/Baxter_isaac/ROS2/src/t42_gripper/t42_g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 scale=0.001 0.001 0.001
- link swivel_2: geometry collision mesh filename=/home/ubb/Documents/Baxter_isaac/ROS2/src/t42_gripper/t42_g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 scale=0.001 0.001 0.001; visual mesh filename=/home/ubb/Documents/Baxter_isaac/ROS2/src/t42_gripper/t42_g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 scale=0.001 0.001 0.001
- link t42_base_link: geometry collision mesh filename=/home/ubb/Documents/Baxter_isaac/ROS2/src/t42_gripper/t42_g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 scale=1 1 1; visual mesh filename=/home/ubb/Documents/Baxter_isaac/ROS2/src/t42_gripper/t42_g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 scale=1 1 1

Commit message: Add arduino to model to prevent collision

File: ur_isaac/urdfs/ur_t42.urdf (robot description, URDF)
Before this commit: robot ur3, 20 links, 19 joints
Links:
- added link arduino_controller; collision mesh filename=/home/ubb/Documents/Baxter_isaac/ROS2/src/t42_gripper/t42_g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; visual mesh filename=/home/ubb/Documents/Baxter_isaac/ROS2/src/t42_gripper/t42_g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
- added link arduino_pc; collision mesh filename=/home/ubb/Documents/Baxter_isaac/ROS2/src/t42_gripper/t42_g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; visual mesh filename=/home/ubb/Documents/Baxter_isaac/ROS2/src/t42_gripper/t42_g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
Joints:
- added joint t42_base_link_to_arduino_controller: type fixed, parent t42_base_link, child arduino_controller, origin xyz=0.02655 0.0 -0.059 rpy=1.57 0 1.57
- added joint t42_base_link_to_arduino_pc: type fixed, parent t42_base_link, child arduino_pc, origin xyz=0.02655 0.0 0.05153 rpy=1.57 0 1.57

Commit message: Update with new safety limit

File: ur_isaac/urdfs/ur_t42.urdf (robot description, URDF)
Before this commit: robot ur3, 22 links, 21 joints
Joints:
- joint shoulder_lift_joint: limit lower=-6.283185307179586 upper=6.283185307179586 effort=56.0 velocity=3.141592653589793 -> lower=-2.35619 upper=-0.79 effort=56.0 velocity=3.141592653589793
- joint wrist_1_joint: limit lower=-6.283185307179586 upper=6.283185307179586 effort=12.0 velocity=6.283185307179586 -> lower=-2.61799 upper=-0.436332 effort=12.0 velocity=6.283185307179586
- joint wrist_2_joint: limit lower=-6.283185307179586 upper=6.283185307179586 effort=12.0 velocity=6.283185307179586 -> lower=-2.61799 upper=2.61799 effort=12.0 velocity=6.283185307179586

Commit message: Add new ee link to reduce possible collision

File: ur_isaac/urdfs/ur_t42.urdf (robot description, URDF)
Before this commit: robot ur3, 22 links, 21 joints
Links:
- added link gripper_ee
Joints:
- added joint t42_base_link_to_gripper_ee: type fixed, parent t42_base_link, child gripper_ee, origin xyz=-0.1 0 0  rpy=0 0 0

Commit message: Update gripper config

File: ur_isaac/urdfs/ur_t42.urdf (robot description, URDF)
Before this commit: robot ur3, 23 links, 22 joints
Links:
- removed link arduino_controller
- removed link arduino_pc
- link t42_base_link: geometry collision mesh filename=/home/ubb/Documents/Baxter_isaac/ROS2/src/t42_gripper/t42_g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 scale=1 1.45 1; visual mesh filename=/home/ubb/Documents/Baxter_isaac/ROS2/src/t42_gripper/t42_g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 scale=1 1.45 1
Joints:
- removed joint t42_base_link_to_arduino_controller
- removed joint t42_base_link_to_arduino_pc
- joint tool_to_gripper: origin xyz=0 0 0.05 rpy=0 1.57 0.785398 -> xyz=0 0 0.09 rpy=0 1.57 0.785398

Commit message: Switch to Real2Sim2Real for controller

File: ur_isaac/urdfs/ur_t42.urdf (robot description, URDF)
Before this commit: robot ur3, 21 links, 20 joints
Links:
- link t42_base_link: geometry collision mesh filename=/home/ubb/Documents/Baxter_isaac/ROS2/src/t42_gripper/t42_g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 scale=1 1.7 1; visual mesh filename=/home/ubb/Documents/Baxter_isaac/ROS2/src/t42_gripper/t42_g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 scale=1 1.7 1
Joints:
- joint shoulder_pan_joint: limit lower=-6.283185307179586 upper=6.283185307179586 effort=56.0 velocity=3.141592653589793 -> lower=-3.23 upper=1.66 effort=56.0 velocity=3.141592653589793
- joint swivel_1_to_finger_1_1: limit lower=0.0 upper=2 effort=10000 velocity=2 -> lower=0.0 upper=3 effort=10000 velocity=2
- joint swivel_2_to_finger_2_1: limit lower=0.0 upper=2 effort=10000 velocity=2 -> lower=0.0 upper=3 effort=10000 velocity=2
- joint t42_base_link_to_gripper_ee: origin xyz=-0.1 0 0  rpy=0 0 0 -> xyz=-0.12 0 0  rpy=0 0 0
- joint tool_to_gripper: origin xyz=0 0 0.09 rpy=0 1.57 0.785398 -> xyz=0 0 0.105 rpy=0 1.57 2.277
- joint wrist_3_joint: limit lower=-6.283185307179586 upper=6.283185307179586 effort=12.0 velocity=6.283185307179586 -> lower=-2.36 upper=4.1 effort=12.0 velocity=6.283185307179586

Commit message: Update Limits

File: ur_isaac/urdfs/ur_t42.urdf (robot description, URDF)
Before this commit: robot ur3, 21 links, 20 joints
Joints:
- joint swivel_1_to_finger_1_1: limit lower=0.0 upper=3 effort=10000 velocity=2 -> lower=0.0 upper=3.1 effort=10000 velocity=2
- joint swivel_2_to_finger_2_1: limit lower=0.0 upper=3 effort=10000 velocity=2 -> lower=0.0 upper=3.1 effort=10000 velocity=2

Commit message: Adjusted limits

File: ur_isaac/urdfs/ur_t42.urdf (robot description, URDF)
Before this commit: robot ur3, 21 links, 20 joints
Joints:
- joint shoulder_pan_joint: limit lower=-3.23 upper=1.66 effort=56.0 velocity=3.141592653589793 -> lower=-3.8 upper=1.57 effort=56.0 velocity=3.141592653589793
- joint tool_to_gripper: origin xyz=0 0 0.105 rpy=0 1.57 2.277 -> xyz=0 0 0.105 rpy=0 1.57 -0.863
- joint wrist_1_joint: limit lower=-2.61799 upper=-0.436332 effort=12.0 velocity=6.283185307179586 -> lower=-1.92 upper=-0.44 effort=12.0 velocity=6.283185307179586

Commit message: Adjusted limits

File: ur_isaac/urdfs/ur_t42.urdf (robot description, URDF)
Before this commit: robot ur3, 21 links, 20 joints
Joints:
- joint elbow_joint: limit lower=-3.141592653589793 upper=3.141592653589793 effort=28.0 velocity=3.141592653589793 -> lower=-2.2 upper=3.141592653589793 effort=28.0 velocity=3.141592653589793
- joint shoulder_lift_joint: limit lower=-2.35619 upper=-0.79 effort=56.0 velocity=3.141592653589793 -> lower=-2.6 upper=-0.79 effort=56.0 velocity=3.141592653589793

Commit message: Bigger limit

File: ur_isaac/urdfs/ur_t42.urdf (robot description, URDF)
Before this commit: robot ur3, 21 links, 20 joints
Joints:
- joint wrist_3_joint: limit lower=-2.36 upper=4.1 effort=12.0 velocity=6.283185307179586 -> lower=-4.1 upper=4.1 effort=12.0 velocity=6.283185307179586

Commit message: Remove hardcoded path

File: ur_isaac/urdfs/ur_t42.urdf (robot description, URDF)
Before this commit: robot ur3, 21 links, 20 joints
Links:
- link finger_1_1: geometry collision mesh filename=package://t42_gripper_description/meshes/proximal_t42.STL scale=0.025400 0.025400 0.025400; visual mesh filename=package://t42_gripper_description/meshes/proximal_t42.STL scale=0.025400 0.025400 0.025400
- link finger_1_2: geometry collision mesh filename=package://t42_gripper_description/meshes/distal_round_t42_f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 scale=0.001 0.001 0.001; visual mesh filename=package://t42_gripper_description/meshes/distal_round_t42_f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 scale=0.001 0.001 0.001
- link finger_2_1: geometry collision mesh filename=package://t42_gripper_description/meshes/proximal_t42.STL scale=0.025400 0.025400 0.025400; visual mesh filename=package://t42_gripper_description/meshes/proximal_t42.STL scale=0.025400 0.025400 0.025400
- link finger_2_2: geometry collision mesh filename=package://t42_gripper_description/meshes/distal_round_t42_f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 scale=0.001 0.001 0.001; visual mesh filename=package://t42_gripper_description/meshes/distal_round_t42_f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 scale=0.001 0.001 0.001
- link swivel_1: geometry collision mesh filename=package://t42_gripper_description/meshes/swivel_t42.STL scale=0.001 0.001 0.001; visual mesh filename=package://t42_gripper_description/meshes/swivel_t42.STL scale=0.001 0.001 0.001
- link swivel_2: geometry collision mesh filename=package://t42_gripper_description/meshes/swivel_t42.STL scale=0.001 0.001 0.001; visual mesh filename=package://t42_gripper_description/meshes/swivel_t42.STL scale=0.001 0.001 0.001
- link t42_base_link: geometry collision mesh filename=package://t42_gripper_description/meshes/actuator_block_t42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 scale=1 1.7 1; visual mesh filename=package://t42_gripper_description/meshes/actuator_block_t42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 scale=1 1.7 1
